File: can-b2b-interconnect.kicad_sch (KiCad schematic)
At the start: 4 parts, among them U5 DF52-4S-0.8H(21)

Commit message: not routed yet, sch
Parts:
- removed U5 (x2): DF52-4S-0.8H(21), can-b2b-interconnect:DF52-4S-0.8H(21), symbol foc-pcb:DF52-4S-0.8H(21)
- added J1, J2: USB4110GFA, can-b2b-interconnect:GCT_USB4105-GF-A, symbol can-b2b-interconnect:USB4110GFA
- added R1 (x2): 5.1k, robot-cortex:R_0402_1005Metric, symbol NeuralStimulatorAndRecorder:Resistor
Connections:
- net CANH: now also J1.A6 (DP1), J1.B6 (DP2), J2.A6 (DP1), J2.B6 (DP2)
- net CANL: now also J1.A7 (DN1), J1.B7 (DN2), J2.A7 (DN1), J2.B7 (DN2)
- net GND: now also J1.A1/B12 (GND), J1.B1/A12 (GND__1), J1.S1 (GND__2), J1.S2 (GND__3), J1.S3 (GND__4), J1.S4 (GND__5), J2.A1/B12 (GND), J2.B1/A12 (GND__1), J2.S1 (GND__2), J2.S2 (GND__3), J2.S3 (GND__4), J2.S4 (GND__5), R1.1, R1.1
- net VBAT: now also J1.A4/B9 (VBUS), J1.B4/A9 (VBUS__1), J2.A4/B9 (VBUS), J2.B4/A9 (VBUS__1)
- new net: J2.A5 (CC1), J2.B5 (CC2), R1.2
- new net: J1.A5 (CC1), J1.B5 (CC2), R1.2
- no-connect marks 0 -> 4
Other:
- moved on the sheet: R1

Commit message: df52 to two usbcs, with optional termination resistor
Parts:
- R1: footprint robot-cortex:R_0402_1005Metric -> can-b2b-interconnect:R_0402_1005Metric
Changed lines of the file:
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@@
       (effects (font (size 1.27 1.27)))
     )
-    (property "Footprint" "robot-cortex:R_0402_1005Metric" (at 132.715 39.37 0)
+    (property "Footprint" "can-b2b-interconnect:R_0402_1005Metric" (at 132.715 39.37 0)
       (effects (font (size 1.27 1.27)) hide)
     )
@@
       (effects (font (size 1.27 1.27)))
     )
-    (property "Footprint" "robot-cortex:R_0402_1005Metric" (at 135.89 92.075 0)
-      (effects (font (size 1.27 1.27)) hide)
-    )
+    (property "Footprint" "can-b2b-interconnect:R_0402_1005Metric" (at 135.89 92.075 0)
+      (effects (font (size 1.27 1.27)) hide)
+    )

Commit message: board designed
Parts:
- removed J1: USB4110GFA, can-b2b-interconnect:GCT_USB4105-GF-A, symbol can-b2b-interconnect:USB4110GFA
- removed R1: 5.1k, can-b2b-interconnect:R_0402_1005Metric, symbol NeuralStimulatorAndRecorder:Resistor
Connections:
- no-connect marks 4 -> 2
