File: can-b2b-interconnect.kicad_pcb (KiCad board)
At the start: 2 copper layers, 6.3 x 13.1 mm, 4 parts, among them U1 DF52-4S-0.8H(21), U2 DF52-4S-0.8H(21), U3 DF52-4S-0.8H(21)

Commit message: updated gnd for panel. updated panel. updated panel script for better more better
Changed lines of the file:
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@@
     (polygon
       (pts
-        (xy 121.61 59.93)
-        (xy 111.98 59.93)
-        (xy 110.92 60.99)
-        (xy 110.92 75.77)
-        (xy 113.11 77.96)
-        (xy 120.67 77.96)
-        (xy 123.9 74.73)
-        (xy 123.9 62.22)
+        (xy 120.32 62.33)
+        (xy 114 62.32)
+        (xy 113.99 75.39)
+        (xy 120.33 75.4)
       )
     )
